File: myProjects/spsu/spsu.brd (EAGLE design)
At the start: 45.7 x 45.7 mm, 21 parts, among them IC1 MC34063A, J1 12V-in, J2 Hi-V, Q1 IRF840, X1 PJ-102A, X2 PJ-102A

Commit message: removed power plugs and replaces with molex added Gerber files
Parts:
- removed X1, X2: PJ-102A, kmarx1:PJ-102-DCJACK
- added J3: 12V, kmarx1:MOLEX-001-2PIN
- J1: value 12V-in -> 12V
Connections:
- net +12V: now also J3.1; no longer X1.1
- net GND: now also J3.2; no longer X1.2, X1.3, X2.2, X2.3
- net HIVOLTAGEOUT: no longer X2.1
Routing:
- net GND: track 119.5 -> 97.2 mm
- net HIVOLTAGEOUT: track 64.9 -> 52.8 mm
- net N$3: track 33.9 -> 24.9 mm
- net +12V: track 87.7 -> 92.1 mm
- net N$4: track 42.3 -> 43.8 mm
- net N$6: track 17.6 -> 16.8 mm
