File: myProjects/ArdLedRing/ArdLedRing.sch (EAGLE design)
At the start: 0 parts

Commit message: finished ArdLedRing design
Parts:
- added C1: 1000 uf, rcl:CPOL-USE3.5-10
- added IC1: PRO-MINI, sibosop:PRO-MINI
- added IC2: SPARKRTC, sibosop:SPARKRTC
- added IC3: 7805, kmarx1:7805
- added U$1: LOGO, sibosop:LOGO
- added U$2, U$3, U$4, U$5: HOLE-125, sibosop:HOLE-125
- added X1: 22-23-2031, sibosop-con-molex:22-23-2031
- added X2: Power, sibosop-con-molex:22-23-2021
- added X4: Minutes, sibosop-con-molex:22-23-2021
- added X5: Hours, sibosop-con-molex:22-23-2021
Connections:
- new net +12V: C1.+, IC3.VI, X2-1.S
- new net GND: C1.-, IC1.GND@1, IC1.GND@2, IC2.GND, IC3.GND, X1-1.S, X2-2.S, X4-2.S, X5-2.S
- new net N$1: IC1.D5, X4-1.S
- new net N$2: IC1.D6, X5-1.S
- new net N$3: IC1.D2, IC2.SQW
- new net N$4: IC1.SCK, IC2.CLK
- new net N$5: IC1.MISO, IC2.MISO
- new net N$6: IC1.MOSI, IC2.MOSI
- new net N$7: IC1.D8, IC2.SS
- new net N$8: IC1.D7, X1-3.S
- new net VCC: IC1.VCC, IC2.VCC, IC3.VO, X1-2.S
